File: Hardware/v4/Arm Board V4.sch (EAGLE design)
At the start: 28 parts, among them P1 STELLARIS-LAUNCHPADSTELLARIS-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, U1 SN74LS241DW, U2 XBEE-1B3

Commit message: okay i think im done reworking arm board
Parts:
- removed D1: RED, SparkFun-LED:LED-RED0603
Connections:
- removed net DDATA_OUT: D1.A, U1.1A1, U1.2Y4
- net DDATA_1: now also U1.1A1, U1.2Y4; no longer D1.C
Changed lines of the file:
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@@
 <part name="GND3" library="SparkFun-Aesthetics" deviceset="GND" device=""/>
 <part name="GND10" library="SparkFun-Aesthetics" deviceset="GND" device=""/>
-<part name="D1" library="SparkFun-LED" deviceset="LED-RED" device="0603" value="RED"/>
 </parts>
 <sheets>
@@
 <instance part="GND3" gate="1" x="198.12" y="17.78" rot="R90"/>
 <instance part="GND10" gate="1" x="162.56" y="7.62" rot="R270"/>
-<instance part="D1" gate="G$1" x="99.06" y="-12.7" rot="R90"/>
 </instances>
 <busses>
@@
 </segment>
 <segment>
-<pinref part="D1" gate="G$1" pin="C"/>
-<wire x1="104.14" y1="-12.7" x2="106.68" y2="-12.7" width="0.1524" layer="91"/>
-<label x="104.14" y="-12.7" size="1.778" layer="95"/>
-</segment>
-</net>
-<net name="RX_1" class="0">
-<segment>
-<pinref part="U1" gate="A" pin="1Y1"/>
-<wire x1="93.98" y1="7.62" x2="99.06" y2="7.62" width="0.1524" layer="91"/>
-<label x="93.98" y="7.62" size="1.778" layer="95"/>
-</segment>
-</net>
-<net name="TX_1" class="0">
-<segment>
-<pinref part="U1" gate="A" pin="2A4"/>
-<wire x1="58.42" y1="-25.4" x2="53.34" y2="-25.4" width="0.1524" layer="91"/>
-<label x="50.8" y="-25.4" size="1.778" layer="95"/>
-</segment>
-</net>
-<net name="TX_3" class="0">
-<segment>
-<pinref part="JP1" gate="G$1" pin="1"/>
-<wire x1="220.98" y1="-25.4" x2="220.98" y2="-33.02" width="0.1524" layer="91"/>
-</segment>
-</net>
-<net name="RX_3" class="0">
-<segment>
-<pinref part="JP1" gate="G$1" pin="2"/>
-<wire x1="223.52" y1="-25.4" x2="223.52" y2="-33.02" width="0.1524" layer="91"/>
-</segment>
-</net>
-<net name="N$9" class="0">
-<segment>
-<pinref part="U$1" gate="G$1" pin="+5V@1"/>
-<wire x1="177.8" y1="25.4" x2="177.8" y2="30.48" width="0.1524" layer="91"/>
-</segment>
-</net>
-<net name="N$11" class="0">
-<segment>
-<pinref part="U$1" gate="G$1" pin="GND@2"/>
-<wire x1="175.26" y1="25.4" x2="175.26" y2="30.48" width="0.1524" layer="91"/>
-</segment>
-</net>
-<net name="N$12" class="0">
-<segment>
-<pinref part="U$1" gate="G$1" pin="FB"/>
-<wire x1="180.34" y1="25.4" x2="180.34" y2="30.48" width="0.1524" layer="91"/>
-</segment>
-</net>
-<net name="RX_7" class="0">
-<segment>
-<pinref part="U$1" gate="G$1" pin="RX"/>
-<wire x1="195.58" y1="12.7" x2="200.66" y2="12.7" width="0.1524" layer="91"/>
-</segment>
-</net>
-<net name="N$21" class="0">
-<segment>
-<pinref part="U$1" gate="G$1" pin="A"/>
-<wire x1="165.1" y1="12.7" x2="160.02" y2="12.7" width="0.1524" layer="91"/>
-</segment>
-</net>
-<net name="N$22" class="0">
-<segment>
-<pinref part="U$1" gate="G$1" pin="B"/>
-<wire x1="165.1" y1="17.78" x2="160.02" y2="17.78" width="0.1524" layer="91"/>
-</segment>
-</net>
-<net name="DDATA_OUT" class="0">
-<segment>
-<pinref part="U1" gate="A" pin="2Y4"/>
-<pinref part="D1" gate="G$1" pin="A"/>
-<wire x1="96.52" y1="-12.7" x2="93.98" y2="-12.7" width="0.1524" layer="91"/>
-<label x="83.82" y="-15.24" size="1.778" layer="95"/>
-</segment>
-<segment>
 <pinref part="U1" gate="A" pin="1A1"/>
 <wire x1="58.42" y1="-5.08" x2="53.34" y2="-5.08" width="0.1524" layer="91"/>
@@
 <wire x1="58.42" y1="-5.08" x2="53.34" y2="-5.08" width="0.1524" layer="91"/>
 </segment>
-</net>
+<segment>
+<pinref part="U1" gate="A" pin="2Y4"/>
+<wire x1="96.52" y1="-12.7" x2="93.98" y2="-12.7" width="0.1524" layer="91"/>
+<label x="83.82" y="-15.24" size="1.778" layer="95"/>
+</segment>
+</net>
+<net name="RX_1" class="0">
+<segment>
+<pinref part="U1" gate="A" pin="1Y1"/>
+<wire x1="93.98" y1="7.62" x2="99.06" y2="7.62" width="0.1524" layer="91"/>
+<label x="93.98" y="7.62" size="1.778" layer="95"/>
+</segment>
+</net>
+<net name="TX_1" class="0">
+<segment>
+<pinref part="U1" gate="A" pin="2A4"/>
+<wire x1="58.42" y1="-25.4" x2="53.34" y2="-25.4" width="0.1524" layer="91"/>
+<label x="50.8" y="-25.4" size="1.778" layer="95"/>
+</segment>
+</net>
+<net name="TX_3" class="0">
+<segment>
+<pinref part="JP1" gate="G$1" pin="1"/>
+<wire x1="220.98" y1="-25.4" x2="220.98" y2="-33.02" width="0.1524" layer="91"/>
+</segment>
+</net>
+<net name="RX_3" class="0">
+<segment>
+<pinref part="JP1" gate="G$1" pin="2"/>
+<wire x1="223.52" y1="-25.4" x2="223.52" y2="-33.02" width="0.1524" layer="91"/>
+</segment>
+</net>
+<net name="N$9" class="0">
+<segment>
+<pinref part="U$1" gate="G$1" pin="+5V@1"/>
+<wire x1="177.8" y1="25.4" x2="177.8" y2="30.48" width="0.1524" layer="91"/>
+</segment>
+</net>
+<net name="N$11" class="0">
+<segment>
+<pinref part="U$1" gate="G$1" pin="GND@2"/>
+<wire x1="175.26" y1="25.4" x2="175.26" y2="30.48" width="0.1524" layer="91"/>
+</segment>
+</net>
+<net name="N$12" class="0">
+<segment>
+<pinref part="U$1" gate="G$1" pin="FB"/>
+<wire x1="180.34" y1="25.4" x2="180.34" y2="30.48" width="0.1524" layer="91"/>
+</segment>
+</net>
+<net name="RX_7" class="0">
+<segment>
+<pinref part="U$1" gate="G$1" pin="RX"/>
+<wire x1="195.58" y1="12.7" x2="200.66" y2="12.7" width="0.1524" layer="91"/>
+</segment>
+</net>
+<net name="N$21" class="0">
+<segment>
+<pinref part="U$1" gate="G$1" pin="A"/>
+<wire x1="165.1" y1="12.7" x2="160.02" y2="12.7" width="0.1524" layer="91"/>
+</segment>
+</net>
+<net name="N$22" class="0">
+<segment>
+<pinref part="U$1" gate="G$1" pin="B"/>
+<wire x1="165.1" y1="17.78" x2="160.02" y2="17.78" width="0.1524" layer="91"/>
+</segment>
+</net>

Commit message: okay now im done
Parts:
- added D1: RED, SparkFun-LED:LED-RED0603
- added R1: 1k, SparkFun-Resistors:RESISTOR1206
Connections:
- new net N$13: D1.A, R1.1
- net +5V: now also R1.2, U$1.+5V_OUT
- net DDATA_1: now also D1.C
Changed lines of the file:
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@@
 <part name="GND3" library="SparkFun-Aesthetics" deviceset="GND" device=""/>
 <part name="GND10" library="SparkFun-Aesthetics" deviceset="GND" device=""/>
+<part name="R1" library="SparkFun-Resistors" deviceset="RESISTOR" device="1206" value="1k"/>
+<part name="D1" library="SparkFun-LED" deviceset="LED-RED" device="0603" value="RED"/>
+<part name="SUPPLY1" library="SparkFun-Aesthetics" deviceset="5V" device=""/>
 </parts>
 <sheets>
@@
 <instance part="GND3" gate="1" x="198.12" y="17.78" rot="R90"/>
 <instance part="GND10" gate="1" x="162.56" y="7.62" rot="R270"/>
+<instance part="R1" gate="G$1" x="22.86" y="17.78" rot="R90"/>
+<instance part="D1" gate="G$1" x="22.86" y="10.16"/>
+<instance part="SUPPLY1" gate="G$1" x="203.2" y="15.24" rot="R270"/>
 </instances>
 <busses>
@@
 <pinref part="U$1" gate="G$1" pin="GND@4"/>
 <pinref part="GND3" gate="1" pin="GND"/>
-<wire x1="193.04" y1="17.78" x2="195.58" y2="17.78" width="0.1524" layer="91"/>
 </segment>
 <segment>
@@
 <wire x1="226.06" y1="-25.4" x2="226.06" y2="-33.02" width="0.1524" layer="91"/>
 <pinref part="JP1" gate="G$1" pin="3"/>
+</segment>
+<segment>
+<pinref part="R1" gate="G$1" pin="2"/>
+<wire x1="22.86" y1="22.86" x2="22.86" y2="25.4" width="0.1524" layer="91"/>
+</segment>
+<segment>
+<pinref part="U$1" gate="G$1" pin="+5V_OUT"/>
+<pinref part="SUPPLY1" gate="G$1" pin="5V"/>
+<wire x1="203.2" y1="15.24" x2="195.58" y2="15.24" width="0.1524" layer="91"/>
 </segment>
 </net>
@@
 <label x="83.82" y="-15.24" size="1.778" layer="95"/>
 </segment>
+<segment>
+<wire x1="22.86" y1="5.08" x2="22.86" y2="2.54" width="0.1524" layer="91"/>
+<pinref part="D1" gate="G$1" pin="C"/>
+</segment>
 </net>
 <net name="RX_1" class="0">
@@
 <pinref part="U$1" gate="G$1" pin="B"/>
 <wire x1="165.1" y1="17.78" x2="160.02" y2="17.78" width="0.1524" layer="91"/>
+</segment>
+</net>
+<net name="N$13" class="0">
+<segment>
+<pinref part="R1" gate="G$1" pin="1"/>
+<pinref part="D1" gate="G$1" pin="A"/>
 </segment>
 </net>
@@
 </schematic>
 </drawing>
-<compatibility>
-<note version="6.3" minversion="6.2.2" severity="warning">
-Since Version 6.2.2 text objects can contain more than one line,
-which will not be processed correctly with this version.
-</note>
-</compatibility>
 </eagle>

Commit message: added refs
added BOM, jrk motor controller ds
Connections:
- net +12V: no longer U$1.VIN
- net GND: no longer U$1.GND@1
Other:
- note removed: "+12V"
Changed lines of the file:
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@@
 <part name="U$1" library="MRDT-RoboticArm" deviceset="TORXIS_BREAKOUT" device=""/>
 <part name="GND3" library="SparkFun-Aesthetics" deviceset="GND" device=""/>
-<part name="GND10" library="SparkFun-Aesthetics" deviceset="GND" device=""/>
 <part name="R1" library="SparkFun-Resistors" deviceset="RESISTOR" device="1206" value="1k"/>
 <part name="D1" library="SparkFun-LED" deviceset="LED-RED" device="0603" value="RED"/>
@@
 <description>Power</description>
 <plain>
-<text x="160.02" y="2.54" size="1.778" layer="95">+12V</text>
 </plain>
 <instances>
@@
 <instance part="U$1" gate="G$1" x="167.64" y="-2.54"/>
 <instance part="GND3" gate="1" x="198.12" y="17.78" rot="R90"/>
-<instance part="GND10" gate="1" x="162.56" y="7.62" rot="R270"/>
 <instance part="R1" gate="G$1" x="22.86" y="17.78" rot="R90"/>
 <instance part="D1" gate="G$1" x="22.86" y="10.16"/>
@@
 <pinref part="GND3" gate="1" pin="GND"/>
 </segment>
-<segment>
-<pinref part="U$1" gate="G$1" pin="GND@1"/>
-<pinref part="GND10" gate="1" pin="GND"/>
-</segment>
 </net>
 <net name="+12V" class="0">
@@
 </segment>
 <segment>
-<pinref part="U$1" gate="G$1" pin="VIN"/>
-<wire x1="165.1" y1="2.54" x2="160.02" y2="2.54" width="0.1524" layer="91"/>
-</segment>
-<segment>

Commit message: arm board
added parts to allow h-bridge actuator drive
Parts:
- added C2: 5.6nF, SparkFun-Passives:CAP1206
- added C4: 220nF, SparkFun-Passives:CAP1206
- added C9: 10nF, SparkFun-Passives:CAP1206
- added D2, D3: 1N4148, SparkFun-DiscreteSemi:DIODE1N4148
- added IC3: L6206D, L6206D:L6206D
- added R15: 100, SparkFun-Resistors:RESISTOR1206
- added R8: 100k, SparkFun-Resistors:RESISTOR1206
- added U$6: H_WR-TBL_3210002VERT, MRDT-2015-PowerBoard:H_WR-TBL_3210002VERT
Connections:
- new net A1: IC3.OUT1_A, U$6.L
- new net A2: IC3.OUT2_A, U$6.R
- new net EN_A: P1.PD2, R8.2
- new net IN1_A: IC3.IN1_A, P1.PD3
- new net N$17: D2.C, D3.A, R15.2
- new net N$18: C9.2, R15.1
- new net N$19: C9.1, IC3.VCP
- new net OCD_A: C2.2, IC3.EN_A, IC3.OCD_A, R8.1
- new net VBOOT: C4.2, D3.C, IC3.VBOOT
- net +12V: now also C4.1, D2.A, IC3.VS_A, IC3.VS_B
- net GND: now also C2.1, IC3.PROGCL_A, IC3.PROGCL_B, IC3.SENSE_A, IC3.SENSE_B
- net IN2_A: now also IC3.IN2_A
Changed lines of the file:
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@@
 <part name="D1" library="SparkFun-LED" deviceset="LED-RED" device="0603" value="RED"/>
 <part name="SUPPLY1" library="SparkFun-Aesthetics" deviceset="5V" device=""/>
+<part name="IC3" library="L6206D" deviceset="L6206" device="D"/>
+<part name="GND17" library="SparkFun-Aesthetics" deviceset="GND" device=""/>
+<part name="GND39" library="SparkFun-Aesthetics" deviceset="GND" device=""/>
+<part name="GND44" library="SparkFun-Aesthetics" deviceset="GND" device=""/>
+<part name="GND46" library="SparkFun-Aesthetics" deviceset="GND" device=""/>
+<part name="R8" library="SparkFun-Resistors" deviceset="RESISTOR" device="1206" value="100k"/>
+<part name="C2" library="SparkFun-Passives" deviceset="CAP" device="1206" value="5.6nF"/>
+<part name="GND47" library="SparkFun-Aesthetics" deviceset="GND" device=""/>
+<part name="D2" library="SparkFun-DiscreteSemi" deviceset="DIODE" device="1N4148" value="1N4148"/>
+<part name="D3" library="SparkFun-DiscreteSemi" deviceset="DIODE" device="1N4148" value="1N4148"/>
+<part name="C4" library="SparkFun-Passives" deviceset="CAP" device="1206" value="220nF"/>
+<part name="C9" library="SparkFun-Passives" deviceset="CAP" device="1206" value="10nF"/>
+<part name="R15" library="SparkFun-Resistors" deviceset="RESISTOR" device="1206" value="100"/>
+<part name="U$6" library="MRDT-2015-PowerBoard" deviceset="H_WR-TBL_32*1*0002" device="VERT"/>
 </parts>
 <sheets>
@@
 <instance part="D1" gate="G$1" x="22.86" y="10.16"/>
 <instance part="SUPPLY1" gate="G$1" x="203.2" y="15.24" rot="R270"/>
+<instance part="U$6" gate="G$1" x="132.08" y="10.16"/>
 </instances>
 <busses>
@@
 <pinref part="R1" gate="G$1" pin="1"/>
 <pinref part="D1" gate="G$1" pin="A"/>
+</segment>
+</net>
+<net name="A1" class="0">
+<segment>
+<pinref part="U$6" gate="G$1" pin="L"/>
+<wire x1="121.92" y1="12.7" x2="116.84" y2="12.7" width="0.1524" layer="91"/>
+<label x="116.84" y="12.7" size="1.778" layer="95"/>
+</segment>
+</net>
+<net name="A2" class="0">
+<segment>
+<pinref part="U$6" gate="G$1" pin="R"/>
+<wire x1="142.24" y1="12.7" x2="147.32" y2="12.7" width="0.1524" layer="91"/>
+<label x="147.32" y="12.7" size="1.778" layer="95"/>
 </segment>
 </net>
@@
 <pinref part="P1" gate="G$1" pin="PE2"/>
 <wire x1="10.16" y1="27.94" x2="5.08" y2="27.94" width="0.1524" layer="91"/>
+<label x="-2.54" y="27.94" size="1.778" layer="95"/>
 </segment>
 </net>
@@
 <pinref part="P1" gate="G$1" pin="PB0"/>
 <wire x1="40.64" y1="78.74" x2="48.26" y2="78.74" width="0.1524" layer="91"/>
+</segment>
+</net>
+<net name="EN_A" class="0">
+<segment>
+<pinref part="P1" gate="G$1" pin="PD2"/>
+<wire x1="40.64" y1="50.8" x2="45.72" y2="50.8" width="0.1524" layer="91"/>
+<label x="45.72" y="50.8" size="1.778" layer="95"/>
+</segment>
+</net>
+<net name="IN1_A" class="0">
+<segment>
+<pinref part="P1" gate="G$1" pin="PD3"/>
+<wire x1="40.64" y1="48.26" x2="45.72" y2="48.26" width="0.1524" layer="91"/>
+<label x="45.72" y="48.26" size="1.778" layer="95"/>
 </segment>
 </net>
@@
 </segment>
 </net>
+</nets>
+</sheet>
+<sheet>
+<description>H-bridge</description>
+<plain>
+</plain>
+<instances>
+<instance part="IC3" gate="G$1" x="40.64" y="45.72"/>
+<instance part="GND17" gate="1" x="15.24" y="55.88" rot="R270"/>
+<instance part="GND39" gate="1" x="15.24" y="38.1" rot="R270"/>
+<instance part="GND44" gate="1" x="58.42" y="60.96" rot="R90"/>
+<instance part="GND46" gate="1" x="58.42" y="33.02" rot="R90"/>
+<instance part="R8" gate="G$1" x="93.98" y="58.42"/>
+<instance part="C2" gate="G$1" x="86.36" y="63.5"/>
+<instance part="GND47" gate="1" x="99.06" y="68.58" rot="R90"/>
+<instance part="D2" gate="G$1" x="81.28" y="45.72" rot="R90"/>
+<instance part="D3" gate="G$1" x="86.36" y="50.8"/>
+<instance part="C4" gate="G$1" x="91.44" y="48.26" rot="R180"/>
+<instance part="C9" gate="G$1" x="66.04" y="55.88" rot="R90"/>
+<instance part="R15" gate="G$1" x="73.66" y="50.8"/>
+</instances>
+<busses>
+</busses>
+<nets>
+<net name="A1" class="0">
+<segment>
+<pinref part="IC3" gate="G$1" pin="OUT1_A"/>
+<wire x1="25.4" y1="50.8" x2="22.86" y2="50.8" width="0.1524" layer="91"/>
+<label x="20.32" y="50.8" size="1.778" layer="95"/>
+</segment>
+</net>
+<net name="A2" class="0">
+<segment>
+<pinref part="IC3" gate="G$1" pin="OUT2_A"/>
+<wire x1="55.88" y1="53.34" x2="58.42" y2="53.34" width="0.1524" layer="91"/>
+<label x="58.42" y="53.34" size="1.778" layer="95"/>
+</segment>
+</net>
+<net name="GND" class="0">
+<segment>
+<pinref part="IC3" gate="G$1" pin="SENSE_A"/>
+<pinref part="GND17" gate="1" pin="GND"/>
+<wire x1="17.78" y1="55.88" x2="25.4" y2="55.88" width="0.1524" layer="91"/>
+</segment>
+<segment>
+<pinref part="IC3" gate="G$1" pin="SENSE_B"/>
+<pinref part="GND39" gate="1" pin="GND"/>
+<wire x1="17.78" y1="38.1" x2="25.4" y2="38.1" width="0.1524" layer="91"/>
+</segment>
+<segment>
+<pinref part="IC3" gate="G$1" pin="PROGCL_A"/>
+<pinref part="GND44" gate="1" pin="GND"/>
+</segment>
+<segment>
+<pinref part="IC3" gate="G$1" pin="PROGCL_B"/>
+<pinref part="GND46" gate="1" pin="GND"/>
+</segment>
+<segment>
+<pinref part="C2" gate="G$1" pin="1"/>
+<pinref part="GND47" gate="1" pin="GND"/>
+<wire x1="96.52" y1="68.58" x2="86.36" y2="68.58" width="0.1524" layer="91"/>
+</segment>
+</net>
+<net name="IN1_A" class="0">
+<segment>
+<pinref part="IC3" gate="G$1" pin="IN1_A"/>
+<wire x1="25.4" y1="60.96" x2="22.86" y2="60.96" width="0.1524" layer="91"/>
+<label x="15.24" y="60.96" size="1.778" layer="95"/>
+</segment>
+</net>
+<net name="IN2_A" class="0">
+<segment>
+<pinref part="IC3" gate="G$1" pin="IN2_A"/>
+<wire x1="25.4" y1="58.42" x2="22.86" y2="58.42" width="0.1524" layer="91"/>
+<label x="15.24" y="58.42" size="1.778" layer="95"/>
+</segment>
+</net>
+<net name="N$17" class="0">
+<segment>
+<pinref part="D2" gate="G$1" pin="C"/>
+<wire x1="81.28" y1="48.26" x2="81.28" y2="50.8" width="0.1524" layer="91"/>
+<pinref part="D3" gate="G$1" pin="A"/>
+<wire x1="81.28" y1="50.8" x2="83.82" y2="50.8" width="0.1524" layer="91"/>
+<pinref part="R15" gate="G$1" pin="2"/>
+<wire x1="78.74" y1="50.8" x2="81.28" y2="50.8" width="0.1524" layer="91"/>
+<junction x="81.28" y="50.8"/>
+</segment>
+</net>
+<net name="N$18" class="0">
+<segment>
+<pinref part="C9" gate="G$1" pin="2"/>
+<pinref part="R15" gate="G$1" pin="1"/>
+<wire x1="68.58" y1="50.8" x2="68.58" y2="55.88" width="0.1524" layer="91"/>
+</segment>
+</net>
+<net name="N$19" class="0">
+<segment>
+<pinref part="C9" gate="G$1" pin="1"/>
+<pinref part="IC3" gate="G$1" pin="VCP"/>
+<wire x1="60.96" y1="55.88" x2="55.88" y2="55.88" width="0.1524" layer="91"/>
+</segment>
+</net>
+<net name="EN_A" class="0">
+<segment>
+<pinref part="R8" gate="G$1" pin="2"/>
+<wire x1="99.06" y1="58.42" x2="101.6" y2="58.42" width="0.1524" layer="91"/>
+<label x="101.6" y="58.42" size="1.778" layer="95"/>
+</segment>
+</net>
+<net name="+12V" class="0">
+<segment>
+<pinref part="C4" gate="G$1" pin="1"/>
+<wire x1="91.44" y1="43.18" x2="81.28" y2="43.18" width="0.1524" layer="91"/>
+<pinref part="D2" gate="G$1" pin="A"/>
+<wire x1="91.44" y1="43.18" x2="101.6" y2="43.18" width="0.1524" layer="91"/>
+<junction x="91.44" y="43.18"/>
+<label x="101.6" y="43.18" size="1.778" layer="95"/>
+<wire x1="81.28" y1="43.18" x2="58.42" y2="43.18" width="0.1524" layer="91"/>
+<pinref part="IC3" gate="G$1" pin="VS_B"/>
+<pinref part="IC3" gate="G$1" pin="VS_A"/>
+<wire x1="58.42" y1="43.18" x2="55.88" y2="43.18" width="0.1524" layer="91"/>
+<wire x1="55.88" y1="50.8" x2="58.42" y2="50.8" width="0.1524" layer="91"/>
+<wire x1="58.42" y1="50.8" x2="58.42" y2="43.18" width="0.1524" layer="91"/>
+<junction x="58.42" y="43.18"/>
+<junction x="81.28" y="43.18"/>
+</segment>
+</net>
+<net name="OCD_A" class="0">
+<segment>
+<pinref part="IC3" gate="G$1" pin="OCD_A"/>
+<wire x1="25.4" y1="53.34" x2="22.86" y2="53.34" width="0.1524" layer="91"/>
+<label x="15.24" y="53.34" size="1.778" layer="95"/>
+</segment>
+<segment>
+<pinref part="R8" gate="G$1" pin="1"/>
+<wire x1="88.9" y1="58.42" x2="86.36" y2="58.42" width="0.1524" layer="91"/>
+<pinref part="C2" gate="G$1" pin="2"/>
+<wire x1="86.36" y1="58.42" x2="86.36" y2="60.96" width="0.1524" layer="91"/>
+<junction x="86.36" y="58.42"/>
+<wire x1="86.36" y1="58.42" x2="86.36" y2="55.88" width="0.1524" layer="91"/>
+<wire x1="86.36" y1="55.88" x2="91.44" y2="55.88" width="0.1524" layer="91"/>
+<label x="91.44" y="55.88" size="1.778" layer="95"/>
+<pinref part="IC3" gate="G$1" pin="EN_A"/>
+<wire x1="86.36" y1="58.42" x2="55.88" y2="58.42" width="0.1524" layer="91"/>
+</segment>
+</net>
+<net name="VBOOT" class="0">
+<segment>
+<pinref part="D3" gate="G$1" pin="C"/>
+<pinref part="C4" gate="G$1" pin="2"/>
+<wire x1="88.9" y1="50.8" x2="91.44" y2="50.8" width="0.1524" layer="91"/>
+<junction x="91.44" y="50.8"/>
+<wire x1="91.44" y1="50.8" x2="101.6" y2="50.8" width="0.1524" layer="91"/>
+<label x="101.6" y="50.8" size="1.778" layer="95"/>
+</segment>
+<segment>
+<pinref part="IC3" gate="G$1" pin="VBOOT"/>
+<wire x1="55.88" y1="38.1" x2="58.42" y2="38.1" width="0.1524" layer="91"/>
+<label x="58.42" y="38.1" size="1.778" layer="95"/>
+</segment>
+</net>
